File: HDMI_to_DB9/HDMI_to_DB9/HDMI_to_DB9.sch (KiCad schematic (older format))
At the start: 22 parts, among them CN1 HDMI- J4, CN2 HDMI- J6, CN3 HDMI- J5, CN4 HDMI- J1, CN5 HDMI- J2, CN6 HDMI- J3, CN7 HDMI- J7, CN8 HDMI- J8, CN9 HDMI- J9, J1 DB9_1, J2 DB9_3, J3 DB9_2, J4 DB9_1, J5 DB9_2, J6 DB9_3, J7 DB9_1, J8 DB9_2, J9 DB9_3

Commit message: Update
Parts:
- removed CN1: HDMI- J4, Connector:HDMI-SMD_A111926-B-01-R_Female, symbol 0My_Library:A111926-A-05-R
- removed CN2: HDMI- J6, Connector:HDMI-SMD_A111926-B-01-R_Female, symbol 0My_Library:A111926-A-05-R
- removed CN3: HDMI- J5, Connector:HDMI-SMD_A111926-B-01-R_Female, symbol 0My_Library:A111926-A-05-R
- removed CN4: HDMI- J1, Connector:HDMI-SMD_A111926-B-01-R_Female, symbol 0My_Library:A111926-A-05-R
- removed CN5: HDMI- J2, Connector:HDMI-SMD_A111926-B-01-R_Female, symbol 0My_Library:A111926-A-05-R
- removed CN6: HDMI- J3, Connector:HDMI-SMD_A111926-B-01-R_Female, symbol 0My_Library:A111926-A-05-R
- removed CN7: HDMI- J7, Connector:HDMI-SMD_A111926-B-01-R_Female, symbol 0My_Library:A111926-A-05-R
- removed CN8: HDMI- J8, Connector:HDMI-SMD_A111926-B-01-R_Female, symbol 0My_Library:A111926-A-05-R
- removed CN9: HDMI- J9, Connector:HDMI-SMD_A111926-B-01-R_Female, symbol 0My_Library:A111926-A-05-R
- removed J1, J4, J7: DB9_1, Connector:DB9_ASSMANN, symbol Connector:DB9_Female
- removed J2, J6, J9: DB9_3, Connector:DB9_ASSMANN, symbol Connector:DB9_Female
- removed J3, J5, J8: DB9_2, Connector:DB9_ASSMANN, symbol Connector:DB9_Female
- added D1, D10, D11, D12, D13, D14, D15, D16, D17, D2, D3, D4, D5, D6, D7, D8, D9: DB9_1, Connector:Vertical_DB9_Female, symbol Connector:DB9_Female
- added J1, J2, J3, J4, J5, J6, J7, J8, J9: HDMI_A, Connector:HDMI-SMD_A111926-B-01-R_Female, symbol 0My_Library:HDMI_A
Connections:
- net GND: now also D1.3, D10.3, D11.3, D12.3, D13.3, D14.3, D15.3, D16.3, D17.3, D2.3, D3.3, D4.3, D5.3, D6.3, D7.3, D8.3, D9.3, J1.17 (GND), J2.17 (GND), J3.17 (GND), J4.17 (GND), J5.17 (GND), J6.17 (GND), J7.17 (GND), J8.17 (GND), J9.17 (GND)
- new net: D14.1, J7.10 (CK+)
- new net: D14.2, J7.12 (CK-)
- new net: D14.6, J7.7 (D0+)
- new net: D14.7, J7.9 (D0-)
- new net: D16.1, J8.10 (CK+)
- new net: D16.2, J8.12 (CK-)
- new net: D16.6, J8.7 (D0+)
- new net: D16.7, J8.9 (D0-)
- new net: D1.1, D1.6, J1.1 (D2+)
- new net: D1.2, D1.7, J1.3 (D2-)
- new net: D3.4, D3.8, J1.10 (CK+)
- new net: D3.5, D3.9, J1.12 (CK-)
- new net: D2.1, D2.6, J1.4 (D1+)
- new net: D2.2, D2.7, J1.6 (D1-)
- new net: D3.1, D3.6, J1.7 (D0+)
- new net: D3.2, D3.7, J1.9 (D0-)
- new net: D4.1, D4.6, J2.1 (D2+)
- new net: D5.6, J2.10 (CK+)
- new net: D5.7, J2.12 (CK-)
- new net: D4.2, D4.7, J2.3 (D2-)
- new net: D4.4, D4.8, J2.4 (D1+)
- new net: D4.5, D4.9, J2.6 (D1-)
- new net: D5.1, J2.7 (D0+)
- new net: D5.2, J2.9 (D0-)
- new net: D5.4, J3.1 (D2+)
- new net: D5.5, J3.3 (D2-)
- new net: D5.8, J3.4 (D1+)
- new net: D5.9, J3.6 (D1-)
- new net: D6.6, J3.10 (CK+)
- new net: D6.7, J3.12 (CK-)
- new net: D6.1, J3.7 (D0+)
- new net: D6.2, J3.9 (D0-)
- new net: D7.1, D7.6, J4.1 (D2+)
- new net: D7.2, D7.7, J4.3 (D2-)
- new net: D9.4, D9.8, J4.10 (CK+)
- new net: D9.5, D9.9, J4.12 (CK-)
- new net: D8.1, D8.6, J4.4 (D1+)
- new net: D8.2, D8.7, J4.6 (D1-)
- new net: D9.1, D9.6, J4.7 (D0+)
- new net: D9.2, D9.7, J4.9 (D0-)
- new net: D10.1, D10.6, J5.1 (D2+)
- new net: D11.6, J5.10 (CK+)
- new net: D11.7, J5.12 (CK-)
- new net: D10.2, D10.7, J5.3 (D2-)
- new net: D10.4, D10.8, J5.4 (D1+)
- new net: D10.5, D10.9, J5.6 (D1-)
- new net: D11.1, J5.7 (D0+)
- new net: D11.2, J5.9 (D0-)
- new net: D11.4, J6.1 (D2+)
- new net: D11.5, J6.3 (D2-)
- new net: D11.8, J6.4 (D1+)
- new net: D11.9, J6.6 (D1-)
- new net: D12.6, J6.10 (CK+)
- new net: D12.7, J6.12 (CK-)
- new net: D12.1, J6.7 (D0+)
- new net: D12.2, J6.9 (D0-)
- new net: D13.6, J7.1 (D2+)
- new net: D13.7, J7.3 (D2-)
- new net: D13.1, J7.4 (D1+)
- new net: D13.2, J7.6 (D1-)
- new net: D15.6, J8.1 (D2+)
- new net: D15.7, J8.3 (D2-)
- new net: D15.1, J8.4 (D1+)
- new net: D15.2, J8.6 (D1-)
- new net: D17.6, J9.1 (D2+)
- new net: D17.4, J9.10 (CK+)
- new net: D17.5, J9.12 (CK-)
- new net: D17.7, J9.3 (D2-)
- new net: D17.1, J9.4 (D1+)
- new net: D17.2, J9.6 (D1-)
- new net: D17.8, J9.7 (D0+)
- new net: D17.9, J9.9 (D0-)
- no-connect marks 135 -> 140
Other:
- note removed: "When I + and V+ are known from sodlering wire to db9_2 connector and rest to db9_3\n"

Commit message: Fixed
Connections:
- net at D16.1: now also J8.7 (D0+); no longer J8.10 (CK+)
- net at D16.2: now also J8.9 (D0-); no longer J8.12 (CK-)
- net at D16.6: now also J8.10 (CK+); no longer J8.7 (D0+)
- net at D16.7: now also J8.12 (CK-); no longer J8.9 (D0-)
- net at J9.1 (D2+): now also D17.1; no longer D17.6
- net at J9.10 (CK+): now also D17.8; no longer D17.4
- net at J9.12 (CK-): now also D17.9; no longer D17.5
- net at J9.3 (D2-): now also D17.2; no longer D17.7
- net at J9.4 (D1+): now also D17.6; no longer D17.1
- net at J9.6 (D1-): now also D17.7; no longer D17.2
- net at J9.7 (D0+): now also D17.4; no longer D17.8
- net at J9.9 (D0-): now also D17.5; no longer D17.9
Changed lines of the file:
@@
 NoConn ~ 8850 7450
 NoConn ~ 8850 7250
-Wire Wire Line
-	8850 7050 9650 7050
-Wire Wire Line
-	8950 6950 8850 6950
-Wire Wire Line
-	8950 6900 8950 6950
-Wire Wire Line
-	9250 6900 8950 6900
-Wire Wire Line
-	9250 6850 9250 6900
-Wire Wire Line
-	9650 6850 9250 6850
-Wire Wire Line
-	9150 6950 9650 6950
-Wire Wire Line
-	9150 6850 9150 6950
-Wire Wire Line
-	8850 6850 9150 6850
-Wire Wire Line
-	8850 6750 9650 6750
-Wire Wire Line
-	9300 6650 8850 6650
-Wire Wire Line
-	9300 6450 9300 6650
-Wire Wire Line
-	9650 6450 9300 6450
-Wire Wire Line
-	8950 6250 9650 6250
-Wire Wire Line
-	8950 6550 8950 6250
-Wire Wire Line
-	8850 6550 8950 6550
-Wire Wire Line
-	9250 6550 9650 6550
-Wire Wire Line
-	9250 6450 9250 6550
-Wire Wire Line
-	8850 6450 9250 6450
-Wire Wire Line
-	9650 6350 8850 6350
 Text Notes 9900 6300 0    50   ~ 0
 I+
@@
 Wire Wire Line
 	10000 4400 9800 4400
-Wire Wire Line
-	9600 4300 10000 4300
-Wire Wire Line
-	10000 4500 9500 4500
 $Comp
 L power:GND #PWR02
@@
 	0    1    1    0
 $EndComp
-Wire Wire Line
-	8950 3900 9800 3900
-Wire Wire Line
-	9800 3900 9800 4400
-Wire Wire Line
-	8950 4000 9900 4000
-Wire Wire Line
-	9900 4000 9900 4600
-Wire Wire Line
-	9900 4600 10000 4600
-Wire Wire Line
-	8950 4100 9600 4100
-Wire Wire Line
-	9600 4100 9600 4300
-Wire Wire Line
-	8950 4200 9500 4200
-Wire Wire Line
-	9500 4200 9500 4500
 NoConn ~ 10000 5100
 NoConn ~ 10000 5000
@@
 NoConn ~ 9950 850
 NoConn ~ 10050 850
+Wire Wire Line
+	8950 3900 9500 3900
+Wire Wire Line
+	9500 3900 9500 4300
+Wire Wire Line
+	9500 4300 10000 4300
+Wire Wire Line
+	8950 4000 9450 4000
+Wire Wire Line
+	9450 4000 9450 4500
+Wire Wire Line
+	9450 4500 10000 4500
+Wire Wire Line
+	8950 4100 9800 4100
+Wire Wire Line
+	9800 4100 9800 4400
+Wire Wire Line
+	8950 4200 9350 4200
+Wire Wire Line
+	9350 4200 9350 4600
+Wire Wire Line
+	9350 4600 10000 4600
+Wire Wire Line
+	8850 6350 9100 6350
+Wire Wire Line
+	9100 6350 9100 6250
+Wire Wire Line
+	9100 6250 9650 6250
+Wire Wire Line
+	8850 6450 9650 6450
+Wire Wire Line
+	9200 6550 9200 6350
+Wire Wire Line
+	9200 6350 9650 6350
+Wire Wire Line
+	8850 6550 9200 6550
+Wire Wire Line
+	8850 6650 9300 6650
+Wire Wire Line
+	9300 6650 9300 6550
+Wire Wire Line
+	9300 6550 9650 6550
+Wire Wire Line
+	8850 6750 9250 6750
+Wire Wire Line
+	9250 6750 9250 6850
+Wire Wire Line
+	9250 6850 9650 6850
+Wire Wire Line
+	8850 6850 9200 6850
+Wire Wire Line
+	9200 6850 9200 7050
+Wire Wire Line
+	9200 7050 9650 7050
+Wire Wire Line
+	9350 6950 9350 6750
+Wire Wire Line
+	9350 6750 9650 6750
+Wire Wire Line
+	8850 6950 9350 6950
+Wire Wire Line
+	8850 7050 9100 7050
+Wire Wire Line
+	9100 7050 9100 7100
+Wire Wire Line
+	9100 7100 9500 7100
+Wire Wire Line
+	9500 7100 9500 6950
+Wire Wire Line
+	9500 6950 9650 6950
 $EndSCHEMATC
