File: MicroD_Stemma_Fanout/Fanout_01/Fanout_01.kicad_pcb (KiCad board)
At the start: 2 copper layers, 34 parts, among them J1 DB25_Male, J10 DB25_Male, J11 Conn_01x04, J12 Conn_01x02, J13 Conn_01x02, J14 Conn_01x02, J15 Conn_01x02, J16 Conn_01x02, J17 Conn_01x02, J18 Conn_01x02, J19 Conn_01x02, J2 Conn_01x02, J20 Conn_01x04, J21 Conn_01x04_Female, J25 DB25_Male, J26 Conn_01x04, J27 Conn_01x02, J28 Conn_01x02, J29 Conn_01x02, J3 Conn_01x04, J30 Conn_01x02, J31 Conn_01x02, J32 Conn_01x02, J33 Conn_01x02, J34 Conn_01x02, J35 Conn_01x04, J4 Conn_01x04, J5 Conn_01x04, J6 Conn_01x04, J7 Conn_01x04, J8 Conn_01x02_Female, J9 Conn_01x04_Female

Commit message: update
Parts:
- moved J13 130.0 mm to (80.5, 17.5), turned to -90 degrees
- moved J30 108.3 mm to (-30.9, 74.9)
- moved J29 104.5 mm to (-39.0, 58.5)
- moved J21 98.5 mm to (15.8, 84.5)
- moved J15 79.1 mm to (-19.5, 58.0), turned to -90 degrees
- moved J28 58.5 mm to (68.8, 27.8)
- moved J27 49.6 mm to (80.2, 23.5)
- moved J12 20.0 mm to (60.8, 15.8)
- moved J11 17.5 mm to (40.2, -7.00)
- moved J20 17.5 mm to (32.2, -7.00)
- moved J26 17.5 mm to (56.2, -7.00)
- moved J3 17.5 mm to (24.2, -7.00)
- moved J35 17.5 mm to (48.2, -7.00)
- moved J4 17.5 mm to (16.2, -7.00)
- moved J5 17.5 mm to (8.25, -7.00)
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