File: Thermometry_MicroD_Adapter/25to25_581/25to25.kicad_sch (KiCad schematic)
At the start: 6 parts, among them J1 Conn_01x02_Male_2.54mm, J2 Conn_01x02_Male_2.54mm, J3 DB25_Male_MountingHoles, J4 DB25_Female_MountingHoles

Commit message: update
fixed 581
Parts:
- removed J? (x2): Conn_01x02_Male_2.54mm, Connector_PinHeader_2.54mm:PinHeader_1x02_P2.54mm_Horizontal, symbol 0JLC-6:Conn_01x02_Male_2.54mm
Connections:
- net GND: now reaches J4.0 (PAD)
- net GND: now also J3.0 (PAD)
Changed lines of the file:
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@@
   (junction (at 133.35 104.14) (diameter 0) (color 0 0 0 0)
   )
-  (junction (at 107.95 109.22) (diameter 0) (color 0 0 0 0)
-  )
-  (junction (at 100.33 99.06) (diameter 0) (color 0 0 0 0)
-  )
   (junction (at 133.35 101.6) (diameter 0) (color 0 0 0 0)
   )
   (junction (at 133.35 96.52) (diameter 0) (color 0 0 0 0)
   )
-  (junction (at 101.219 96.52) (diameter 0) (color 0 0 0 0)
-  )
-  (junction (at 105.41 106.68) (diameter 0) (color 0 0 0 0)
-  )
-  (wire (pts (xy 105.41 116.459) (xy 105.41 106.68))
-    (stroke (width 0) (type default) (color 0 0 0 0))
-  )
-  (wire (pts (xy 95.25 96.52) (xy 101.219 96.52))
-    (stroke (width 0) (type default) (color 0 0 0 0))
-  )
-  (wire (pts (xy 107.95 109.22) (xy 107.95 118.999))
-    (stroke (width 0) (type default) (color 0 0 0 0))
-  )
   (wire (pts (xy 105.41 106.68) (xy 105.41 101.6))
     (stroke (width 0) (type default) (color 0 0 0 0))
   )
-  (wire (pts (xy 95.25 99.06) (xy 100.33 99.06))
-    (stroke (width 0) (type default) (color 0 0 0 0))
-  )
-  (wire (pts (xy 100.33 89.027) (xy 100.33 99.06))
-    (stroke (width 0) (type default) (color 0 0 0 0))
-  )
-  (wire (pts (xy 95.25 116.459) (xy 105.41 116.459))
-    (stroke (width 0) (type default) (color 0 0 0 0))
-  )
-  (wire (pts (xy 94.361 86.487) (xy 101.219 86.487))
+  (wire (pts (xy 95.25 99.06) (xy 133.35 99.06))
     (stroke (width 0) (type default) (color 0 0 0 0))
   )
@@
     (stroke (width 0) (type default) (color 0 0 0 0))
   )
-  (wire (pts (xy 94.361 89.027) (xy 100.33 89.027))
-    (stroke (width 0) (type default) (color 0 0 0 0))
-  )
-  (wire (pts (xy 100.33 99.06) (xy 133.35 99.06))
-    (stroke (width 0) (type default) (color 0 0 0 0))
-  )
   (wire (pts (xy 107.95 109.22) (xy 95.25 109.22))
     (stroke (width 0) (type default) (color 0 0 0 0))
@@
     (stroke (width 0) (type default) (color 0 0 0 0))
   )
-  (wire (pts (xy 107.95 118.999) (xy 95.25 118.999))
-    (stroke (width 0) (type default) (color 0 0 0 0))
-  )
-  (wire (pts (xy 101.219 96.52) (xy 133.35 96.52))
+  (wire (pts (xy 95.25 96.52) (xy 133.35 96.52))
     (stroke (width 0) (type default) (color 0 0 0 0))
   )
@@
     (stroke (width 0) (type default) (color 0 0 0 0))
   )
-  (wire (pts (xy 101.219 86.487) (xy 101.219 96.52))
-    (stroke (width 0) (type default) (color 0 0 0 0))
-  )
   (wire (pts (xy 95.25 106.68) (xy 105.41 106.68))
     (stroke (width 0) (type default) (color 0 0 0 0))
+  )
+  (symbol (lib_id "power:GND") (at 125.73 50.8 180) (unit 1)
+    (in_bom yes) (on_board yes) (fields_autoplaced)
+    (property "Reference" "#PWR0102" (id 0) (at 125.73 44.45 0)
+      (effects (font (size 1.27 1.27)) hide)
+    )
+    (property "Value" "GND" (id 1) (at 125.73 47.2242 0))
+    (property "Footprint" "" (id 2) (at 125.73 50.8 0)
+      (effects (font (size 1.27 1.27)) hide)
+    )
+    (property "Datasheet" "" (id 3) (at 125.73 50.8 0)
+      (effects (font (size 1.27 1.27)) hide)
+    )
+    (pin "1")
   )
   (symbol (lib_id "0JLC-6:Conn_01x02_Male_2.54mm") (at 90.17 96.52 0) (unit 1)
@@
     (pin "9")
   )
-  (symbol (lib_id "0JLC-6:Conn_01x02_Male_2.54mm") (at 89.281 86.487 0) (unit 1)
-    (in_bom yes) (on_board yes) (fields_autoplaced)
-    (property "Reference" "J?" (id 0) (at 89.916 81.407 0))
-    (property "Value" "Conn_01x02_Male_2.54mm" (id 1) (at 89.916 83.947 0))
-    (property "Footprint" "Connector_PinHeader_2.54mm:PinHeader_1x02_P2.54mm_Horizontal" (id 2) (at 89.281 86.487 0)
-      (effects (font (size 1.27 1.27)) hide)
-    )
-    (property "Datasheet" "~" (id 3) (at 89.281 86.487 0)
-      (effects (font (size 1.27 1.27)) hide)
-    )
-    (property "LCSC" "C492401" (id 4) (at 89.281 86.487 0)
-      (effects (font (size 1.27 1.27)) hide)
-    )
-    (property "MPN" "PZ254V-11-02P" (id 5) (at 89.281 86.487 0)
-      (effects (font (size 1.27 1.27)) hide)
-    )
-    (pin "1")
-    (pin "2")
-  )
-  (symbol (lib_id "0JLC-6:Conn_01x02_Male_2.54mm") (at 90.17 116.459 0) (unit 1)
-    (in_bom yes) (on_board yes) (fields_autoplaced)
-    (property "Reference" "J?" (id 0) (at 90.805 111.379 0))
-    (property "Value" "Conn_01x02_Male_2.54mm" (id 1) (at 90.805 113.919 0))
-    (property "Footprint" "Connector_PinHeader_2.54mm:PinHeader_1x02_P2.54mm_Horizontal" (id 2) (at 90.17 116.459 0)
-      (effects (font (size 1.27 1.27)) hide)
-    )
-    (property "Datasheet" "~" (id 3) (at 90.17 116.459 0)
-      (effects (font (size 1.27 1.27)) hide)
-    )
-    (property "LCSC" "C492401" (id 4) (at 90.17 116.459 0)
-      (effects (font (size 1.27 1.27)) hide)
-    )
-    (property "MPN" "PZ254V-11-02P" (id 5) (at 90.17 116.459 0)
-      (effects (font (size 1.27 1.27)) hide)
-    )
-    (pin "1")
-    (pin "2")
+  (symbol (lib_id "power:GND") (at 140.97 121.92 0) (unit 1)
+    (in_bom yes) (on_board yes) (fields_autoplaced)
+    (property "Reference" "#PWR0101" (id 0) (at 140.97 128.27 0)
+      (effects (font (size 1.27 1.27)) hide)
+    )
+    (property "Value" "GND" (id 1) (at 140.97 126.3634 0))
+    (property "Footprint" "" (id 2) (at 140.97 121.92 0)
+      (effects (font (size 1.27 1.27)) hide)
+    )
+    (property "Datasheet" "" (id 3) (at 140.97 121.92 0)
+      (effects (font (size 1.27 1.27)) hide)
+    )
+    (pin "1")
   )
   (symbol (lib_id "Connector:DB25_Male_MountingHoles") (at 125.73 86.36 180) (unit 1)
@@
   )
   (symbol_instances
+    (path "/936b49d2-308c-40ca-b941-110ed638bd0e"
+      (reference "#PWR0101") (unit 1) (value "GND") (footprint "")
+    )
+    (path "/169a7d34-93e8-4b65-ab2f-e746ccf1ce23"
+      (reference "#PWR0102") (unit 1) (value "GND") (footprint "")
+    )
     (path "/2b2837a2-64fc-46b1-9f8c-1c4dc0037ed3"
       (reference "J1") (unit 1) (value "Conn_01x02_Male_2.54mm") (footprint "Connector_PinHeader_2.54mm:PinHeader_1x02_P2.54mm_Horizontal")
@@
       (reference "J4") (unit 1) (value "DB25_Female_MountingHoles") (footprint "0Project_Library:581M25213L461_Norcomp_Female")
     )
-    (path "/94ed6b35-a22f-4041-976c-2fb459de60b2"
-      (reference "J?") (unit 1) (value "Conn_01x02_Male_2.54mm") (footprint "Connector_PinHeader_2.54mm:PinHeader_1x02_P2.54mm_Horizontal")
-    )
-    (path "/ab18258a-69d7-438b-8679-e87dab86b2a8"
-      (reference "J?") (unit 1) (value "Conn_01x02_Male_2.54mm") (footprint "Connector_PinHeader_2.54mm:PinHeader_1x02_P2.54mm_Horizontal")
-    )
-  )
+  )
