File: Thermometry_MicroD_Adapter/25to25_581/25to25.kicad_pcb (KiCad board)
At the start: 2 copper layers, 65 x 24.3 mm, 6 parts, among them J1 Conn_01x02_Male_2.54mm, J2 Conn_01x02_Male_2.54mm, J3 DB25_Male_MountingHoles, J4 DB25_Female_MountingHoles, J5 Conn_01x02_Male_2.54mm, J6 Conn_01x02_Male_2.54mm

Commit message: update
fixed 581
Parts:
- removed J5, J6: Conn_01x02_Male_2.54mm, Connector_PinHeader_2.54mm:PinHeader_1x02_P2.54mm_Horizontal
- moved J1 8.60 mm to (119.3, 62.8)
- moved J4 6.20 mm to (157.0, 79.5)
- moved J2 0.63 mm to (126.7, 62.8)
Connections:
- J3 pad 0: unconnected-(J3-Pad0) -> GND
- J4 pad 0: unconnected-(J4-Pad0) -> GND
Routing:
- net Net-(J1-Pad1): track 58.4 -> 45.8 mm
- net Net-(J1-Pad2): track 57.0 -> 44.9 mm
- net Net-(J2-Pad1): track 44.3 -> 36.1 mm
- net Net-(J3-Pad8): track 5.65 -> 11.9 mm
- net Net-(J3-Pad7): track 5.65 -> 11.9 mm
- net Net-(J3-Pad6): track 5.65 -> 11.9 mm
- net Net-(J3-Pad5): track 5.65 -> 11.9 mm
- net Net-(J3-Pad4): track 5.65 -> 11.9 mm
- net Net-(J3-Pad3): track 5.65 -> 11.9 mm
- net Net-(J3-Pad2): track 5.65 -> 11.9 mm
- net Net-(J3-Pad13): track 5.65 -> 11.9 mm
- net Net-(J3-Pad12): track 5.65 -> 11.9 mm
- net Net-(J3-Pad11): track 5.65 -> 11.9 mm
- net Net-(J3-Pad1): track 5.65 -> 11.9 mm
- net Net-(J3-Pad25): track 10.7 -> 16.9 mm
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- added copper zone on B.Cu, net GND
- added copper zone on F.Cu, net GND
Other:
- board size 65 x 24.3 mm -> 48.9 x 30.6 mm
