File: KF40_DB25_PinHeader/KF40_DB25_Pinheader/KF40_DB25_Pinheader.kicad_pcb (KiCad board)
At the start: 4 copper layers, 75 x 113.1 mm, 14 parts, among them J1 DB25_Plug, J2 Conn_01x04_Socket, J3 Conn_01x04_Socket, J4 Conn_01x04_Socket, J5 Conn_01x04_Socket, J6 Conn_01x04_Socket, J7 Conn_01x02_Socket, J8 Conn_01x02_Socket

Commit message: update
Other:
- board size 75 x 113.1 mm -> 75 x 102.1 mm
Changed lines of the file:
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@@
   (gr_circle (center 0 0) (end 20.6 0)
     (stroke (width 0.2) (type solid)) (fill none) (layer "Dwgs.User"))
-  (gr_line (start 27.5 -75.6) (end 27.5 -25.5)
+  (gr_line (start 27.5 -64.6) (end 27.5 -25.5)
     (stroke (width 0.2) (type solid)) (layer "Edge.Cuts"))
-  (gr_line (start -27.5 -75.6) (end 27.5 -75.6)
+  (gr_line (start -27.5 -64.6) (end 27.5 -64.6)
     (stroke (width 0.2) (type solid)) (layer "Edge.Cuts"))
   (gr_arc (start 27.5 -25.5) (mid 0 37.503333) (end -27.5 -25.5)
     (stroke (width 0.1) (type default)) (layer "Edge.Cuts"))
-  (gr_line (start -27.5 -25.5) (end -27.5 -75.6)
+  (gr_line (start -27.5 -25.5) (end -27.5 -64.6)
     (stroke (width 0.2) (type solid)) (layer "Edge.Cuts"))
   (segment (start 16.62 -53.58) (end 16.62 -6.36) (width 0.1) (layer "In1.Cu") (net 2))
